Commit message: camera added to end effector for iiwa7

File: iiwa_description/urdf/iiwa7.urdf.xacro (robot description, xacro)
@@ -5,4 +5,5 @@
   <!--Import the lbr iiwa macro -->
   <xacro:include filename="$(find iiwa_description)/urdf/iiwa7.xacro"/>
+  <xacro:property name="camera_link" value="0.1" /> <!-- Size of square 'camera' box -->
   <xacro:arg name="hardware_interface" default="PositionJointInterface"/>
   <xacro:arg name="robot_name" default="iiwa"/>
@@ -15,3 +16,70 @@
     <origin xyz="$(arg origin_xyz)" rpy="$(arg origin_rpy)" />
   </xacro:iiwa7>
+  <joint name="camera_joint" type="fixed">
+    <origin xyz="0 0 00.0500001" rpy="0 -1.57 0"/>
+    <axis xyz="0 0 1"/>
+    <parent link="iiwa_link_ee"/>
+    <child link="camera_link"/>
+  </joint>
+	  <!-- Camera -->
+  <link name="camera_link">
+    <collision>
+      <origin xyz="0 0 0" rpy="0 0 0"/>
+      <geometry>
+    <box size="${camera_link} ${camera_link} ${camera_link}"/>
+      </geometry>
+    </collision>
+    <visual>
+      <origin xyz="00 0 0" rpy="0 0 0"/>
+      <geometry>
+    <box size="${camera_link} ${camera_link} ${camera_link}"/>
+      </geometry>
+      <material name="red"/>
+    </visual>
+    <inertial>
+      <mass value="1e-5" />
+      <origin xyz="0 0 0" rpy="0 0 0"/>
+      <inertia ixx="1e-6" ixy="0" ixz="0" iyy="1e-6" iyz="0" izz="1e-6" />
+    </inertial>
+  </link>
+	<!-- camera -->
+  <gazebo reference="camera_link">
+    <sensor type="camera" name="camera1">
+      <update_rate>30.0</update_rate>
+      <camera name="head">
+        <horizontal_fov>1.3962634</horizontal_fov>
+        <image>
+          <width>800</width>
+          <height>800</height>
+          <format>R8G8B8</format>
+        </image>
+        <clip>
+          <near>0.02</near>
+          <far>300</far>
+        </clip>
+        <noise>
+          <type>gaussian</type>
+          <!-- Noise is sampled independently per pixel on each frame.
+               That pixel's noise value is added to each of its color
+               channels, which at that point lie in the range [0,1]. -->
+          <mean>0.0</mean>
+          <stddev>0.007</stddev>
+        </noise>
+      </camera>
+      <plugin name="camera_controller" filename="libgazebo_ros_camera.so">
+        <alwaysOn>true</alwaysOn>
+        <updateRate>0.0</updateRate>
+        <cameraName>rrbot/camera1</cameraName>
+        <imageTopicName>image_raw</imageTopicName>
+        <cameraInfoTopicName>camera_info</cameraInfoTopicName>
+        <frameName>camera_link</frameName>
+        <hackBaseline>0.07</hackBaseline>
+        <distortionK1>0.0</distortionK1>
+        <distortionK2>0.0</distortionK2>
+        <distortionK3>0.0</distortionK3>
+        <distortionT1>0.0</distortionT1>
+        <distortionT2>0.0</distortionT2>
+      </plugin>
+    </sensor>
+  </gazebo>
 </robot>

File: iiwa_description/urdf/iiwa7.xacro (robot description, xacro)
@@ -293,14 +293,4 @@
     <link name="${robot_name}_link_ee">
     </link>
-        <gazebo>
-          <plugin name="gazebo_ros_vacuum_gripper" filename="libgazebo_ros_vacuum_gripper.so">
-            <robotNamespace>/${robot_name}/vacuum_gripper</robotNamespace>
-            <bodyName>${robot_name}_link_ee</bodyName>
-            <topicName>grasping</topicName>
-            <maxForce>200</maxForce>
-            <maxDistance>10</maxDistance>
-            <minDistance>0</minDistance>
-          </plugin>
-        </gazebo>
     <!--Extensions -->
     <xacro:iiwa_gazebo robot_name="${robot_name}" />

Commit message: Completed Task 1-14 for Kuka_IIWA_Kitting_Cell Project. Added vacuum gripper to the manipulator. https://github.com/bharatm11/Kuka_IIWA_Kitting_Cell

File: iiwa_description/urdf/iiwa7.urdf.xacro (robot description, xacro)
@@ -9,4 +9,5 @@
   <xacro:arg name="origin_xyz" default="0 0 0"/>
   <xacro:arg name="origin_rpy" default="0 0 0"/>
+  <xacro:property name="camera_link" value="0.1" /> <!-- Size of square 'camera' box -->
   <!-- Fix to world just for testing -->
   <link name="world"/>
@@ -15,3 +16,41 @@
     <origin xyz="$(arg origin_xyz)" rpy="$(arg origin_rpy)" />
   </xacro:iiwa7>
+  <!--**********************************-->
+  <joint name="iiwa_camera_joint" type="revolute">
+    <origin xyz="0 0 00.100001" rpy="0 -1.57 0"/>
+    <axis xyz="0 0 1"/>
+    <limit effort="1000.0" lower="0" upper="0" velocity="0"/>
+    <parent link="iiwa_link_7"/>
+    <child link="iiwa_camera_link"/>
+  </joint>
+  <!--**********************************-->
+  <link name="iiwa_camera_link">
+    <!--<collision>
+      <origin xyz="0 0 0" rpy="0 0 0"/>
+      <geometry>
+        <box size="${camera_link} ${camera_link} ${camera_link}"/>
+      </geometry>
+    </collision>-->
+    <visual>
+      <origin xyz="00 0 0" rpy="0 0 0"/>
+      <geometry>
+        <box size="${camera_link} ${camera_link} ${camera_link}"/>
+      </geometry>
+      <material name="red"/>
+    </visual>
+    <inertial>
+      <mass value="1e-5" />
+      <origin xyz="0 0 0" rpy="0 0 0"/>
+      <inertia ixx="1e-6" ixy="0" ixz="0" iyy="1e-6" iyz="0" izz="1e-6" />
+    </inertial>
+  </link>
+  <!--**********************************-->
+  <gazebo>
+      <plugin name="gazebo_ros_vacuum_gripper" filename="libgazebo_ros_vacuum_gripper.so">
+        <robotNamespace>/robot/left_vacuum_gripper</robotNamespace>
+        <bodyName>iiwa_camera_link</bodyName>
+        <topicName>grasping</topicName>
+      </plugin>
+    </gazebo>
+<!--**********************************-->
 </robot>

File: iiwa_description/urdf/iiwa7.xacro (robot description, xacro)
@@ -293,14 +293,4 @@
     <link name="${robot_name}_link_ee">
     </link>
-        <gazebo>
-          <plugin name="gazebo_ros_vacuum_gripper" filename="libgazebo_ros_vacuum_gripper.so">
-            <robotNamespace>/${robot_name}/vacuum_gripper</robotNamespace>
-            <bodyName>${robot_name}_link_ee</bodyName>
-            <topicName>grasping</topicName>
-            <maxForce>200</maxForce>
-            <maxDistance>10</maxDistance>
-            <minDistance>0</minDistance>
-          </plugin>
-        </gazebo>
     <!--Extensions -->
     <xacro:iiwa_gazebo robot_name="${robot_name}" />
